Commit message: fdg

File: husky_group/urdf/husky_urdf_extras.urdf (robot description, URDF)
Before this commit: robot None, 2 links, 2 joints
Joints:
- joint lidar_joint: origin xyz=-0.0635 0 0.610 rpy=0 0 0 -> xyz=-0.0635 0 0.610 rpy=0 0 {pi}

Commit message: khjghj

File: husky_group/urdf/husky_urdf_extras.urdf (robot description, URDF)
Before this commit: robot None, 2 links, 2 joints
Joints:
- joint lidar_joint: origin xyz=-0.0635 0 0.610 rpy=0 0 {pi} -> xyz=-0.0635 0 0.610 rpy=0 0 0

Commit message: pi?

File: husky_group/urdf/husky_urdf_extras.urdf (robot description, URDF)
Before this commit: robot None, 2 links, 2 joints
Joints:
- joint lidar_joint: origin xyz=-0.0635 0 0.610 rpy=0 0 0 -> xyz=-0.0635 0 0.610 rpy=0 0 {$pi}

Commit message: pi!

File: husky_group/urdf/husky_urdf_extras.urdf (robot description, URDF)
Before this commit: robot None, 2 links, 2 joints
Joints:
- joint lidar_joint: origin xyz=-0.0635 0 0.610 rpy=0 0 {$pi} -> xyz=-0.0635 0 0.610 rpy=0 0 3.14159
