Commit message: gdsfgdsgf

File: husky_group/urdf/sim_husky_urdf_extras.urdf (robot description, URDF)
Before this commit: robot None, 2 links, 2 joints
Links:
- link frame_link: geometry collision mesh filename=file://$(find husky_group)/meshes/frame_link.STL; visual mesh filename=file://$(find husky_group)/meshes/frame_link.STL
Joints:
- joint lidar_joint: origin xyz=-0.0635 0 0.610 rpy=0 0 0 -> xyz=-0.0635 0 0.610 rpy=0 0 3.14159

Commit message: sim changes

File: husky_group/urdf/sim_husky_urdf_extras.urdf (robot description, URDF)
Before this commit: robot None, 2 links, 2 joints
Links:
- link frame_link: geometry collision mesh filename=file://$(find husky_group)meshes/frame_link.STL; visual mesh filename=file://$(find husky_group)/meshes/frame_link.STL
